File: EntireBoard/entireboard_v1.sch (EAGLE design)
At the start: 26 parts, among them U2 RHD2216_QFN

Commit message: add connector, crystals, bom, lbr
Parts:
- added 38.768KHZ: EPSON_32.768KHZ_CRYSTAL, AxonMobile:EPSON_32.768KHZ_CRYSTAL
- added 48MHZ: NDK_48MHZ_CRYSTAL, AxonMobile:NDK_48MHZ_CRYSTAL
- added C18, C19: 12pF, adafruit:C-USC0402
- added C20: 0.1uF, adafruit:C-USC0402
- added J1: FTSH-105-01-XXX-DV-K, AxonMobile:FTSH-105-01-XXX-DV-K
- added R1: 100k, AxonMobile:R-US_R0402
- L1, L3, L4, L5, L6: device rcl:L-US0204/5 -> AxonMobile:L-SMD
Connections:
- removed net DIO5/JTAG_TDO: CC2652R1.DIO_5
- removed net DIO6/JTAG_TDI: CC2652R1.DIO_6
- new net JTAG_TDI: CC2652R1.DIO_17, J1.8
- new net JTAG_TDO: CC2652R1.DIO_16, J1.6
- new net N$10: 38.768KHZ.P$2, C19.1, CC2652R1.X32K_Q2
- new net N$3: 48MHZ.P$1, CC2652R1.X48M_P
- new net N$4: 48MHZ.P$2, CC2652R1.X48M_N
- new net N$5: 38.768KHZ.P$1, C18.1, CC2652R1.X32K_Q1
- new net WMCU_RESET: C20.1, CC2652R1.RESET_N, J1.10, R1.1
- net GND: now also 48MHZ.P$GND1, 48MHZ.P$GND2, C17.2, C18.2, C19.2, C20.2, CC2652R1.EGP, J1.3, J1.5, J1.9; no longer C17.1, CC2652R1.ETP
- net JTAG_TCK: now also J1.4
- net JTAG_TMS: now also J1.2
- net N$1: now also C17.1; no longer C17.2
- net VDDS: now also R1.2
Other:
- note added: "JTAG Debugging Connector"
- note added: "TODO: add 0ohm resistor for rebustness"
- moved on the sheet: C11, C12, C13, C14, C15, C16, C17, L3, L4, L5, L6

Commit message: add headers, testpads, current sense resistors, led
Parts:
- added 3.3V, GND: MF-CON-2.54mm-01x01, AxonMobile:CON_01X01_PTH_2.54MM
- added BTN_RESET: SW_1188E, AxonMobile:SW_1188E
- added CURRENT-SENSE, R_CS: 0.01ohm, MF_Passives:RESISTOR_0402
- added POWER_IND: LED-SMD, AxonMobile:LED-SMD
- added R2: (no value), AxonMobile:R-US_R0402
- added TP_SPI_CLK, TP_SPI_CS, TP_SPI_MISO, TP_SPI_MOSI: RHD2000_EVAL_BOARD_TESTPOINT_SMALL, AxonMobile:RHD2000_EVAL_BOARD_TESTPOINT_SMALL
Connections:
- removed net SPI_CS: CC2652R1.DIO_7, U2.!CS!+
- new net N$11: C11.2, CURRENT-SENSE.P$1
- new net N$13: POWER_IND.A, R_CS.P$2
- new net N$16: BTN_RESET.P$4, R2.2
- new net SPI_CS_TP: CC2652R1.DIO_7, TP_SPI_CS.1, U2.!CS!+
- net GND: now also BTN_RESET.P$1, BTN_RESET.P$2, BTN_RESET.P$3, GND.PIN1
- net N$2: now also CURRENT-SENSE.P$2; no longer C11.2
- net SPI_CLK: now also TP_SPI_CLK.1
- net SPI_MISO: now also TP_SPI_MISO.1
- net SPI_MOSI: now also TP_SPI_MOSI.1
- net VDDS: now also POWER_IND.C, R_CS.P$1
- net WMCU_RESET: now also R2.1
- net WMCU_VDD: now also 3.3V.PIN1
Other:
- note added: "3.3V Ext Supply"
- note added: "5V Ext Supply"
- note added: "GND Pin"
- note added: "NOTE: add pads on 4 SPI signal lines for testing"
- note removed: "TODO: add 0ohm resistor for rebustness"
- moved on the sheet: C20, R1
