File: EntireBoard/entireboard_v3.sch (EAGLE design)
At the start: 52 parts, among them J1 FTSH-105-01-XXX-DV-K, P1 0532610271, U1 TPS7A0533PYKAR, U2 RHD2216_QFN

Commit message: modify schematics, changed parts
Parts:
- removed L7: AIML-0603-6R8K-T, inductor_0603:AIML-0603-6R8K-T
- removed POWER_IND: LED-SMD, AxonMobile:LED-SMD
- removed R_CS: 0.01ohm, MF_Passives:RESISTOR_0402
- added L6: 6.8uH, MF_Passives:INDUCTOR_0603
- C6, C8: device adafruit:C-USC0402 -> MF_Passives:CAPACITOR_NP_0603
- J1: value FTSH-105-01-XXX-DV-K -> MF-CON-2.54mm-01x09; device AxonMobile:FTSH-105-01-XXX-DV-K -> MF_Connectors:CON_01X09_PTH_2.54MM
- U1: value TPS7A0533PYKAR -> TPS7A0508PDBVRDBV0005A_M; device yka0004:TPS7A0533PYKAR -> yka0004:TPS7A0508PDBVRDBV0005A_M
Connections:
- removed net N$13: POWER_IND.A, R_CS.P$2
- removed net VDDS: C3.1, C4.1, C5.1, C6.1, C7.1, CC2652R1.VDDS, CC2652R1.VDDS2, CC2652R1.VDDS3, CC2652R1.VDDS_DCDC, L2.2, POWER_IND.C, R1.2, R_CS.P$1
- new net RXD: J1.PIN3
- new net TXD: J1.PIN4
- new net VDDS3V3: C3.1, C4.1, C5.1, C6.P$1, C7.1, CC2652R1.VDDS, CC2652R1.VDDS2, CC2652R1.VDDS3, CC2652R1.VDDS_DCDC, J1.PIN2, L2.2, R1.2
- net DCDC_SW: now also L6.P$1; no longer L7.2
- net GND: now also C6.P$2, C8.P$2, J1.PIN1; no longer C6.2, C8.2, J1.3, J1.5, J1.9
- net JTAG_TCK: now also J1.PIN7; no longer J1.4
- net JTAG_TDI: now also J1.PIN9; no longer J1.8
- net JTAG_TDO: now also J1.PIN8; no longer J1.6
- net JTAG_TMS: now also J1.PIN6; no longer J1.2
- net VDDR: now also C8.P$1, L6.P$2; no longer C8.1, L7.1
- net WMCU_RESET: now also J1.PIN5; no longer J1.10
Other:
- note added: "3V3"
- note added: "GND"
- note added: "RESET"
- note added: "RXD"
- note added: "TCK"
- note added: "TDI"
- note added: "TDO"
- note added: "TMS"
- note added: "TXD"
