File: EntireBoard/entireboard_v3.brd (EAGLE design)
At the start: 40 x 40 mm, 50 parts, among them J2 MF-CON-2.54mm-01x05, J3 MF-CON-2.54mm-01x04, P1 0532610271, U1 TPS7A0508PDBVRDBV0005A_M, U2 RHD2216_QFN

Commit message: final (??) board v3
Parts:
- removed CC2652R1: CC2652R1, AxonMobile:CC2652R1_QFN-48
- added J1, J4: MF-CON-2.54mm-01x05, MF_Connectors:PTH_2.54MM_01X05
- added U$1: CC2652R1, AxonMobile:CC2652R1_QFN-48
- moved SPI_MISO 8.12 mm to (29.2, 31.5)
- moved SPI_MOSI 8.12 mm to (31.0, 31.5)
- moved SPI_CLK 8.12 mm to (32.8, 31.5)
- moved SPI_CS 8.12 mm to (34.6, 31.5)
- moved C1 4.68 mm to (28.8, 28.2)
- moved U2 4.68 mm to (32.2, 22.0)
- moved C2 3.45 mm to (26.0, 25.0)
- moved C18 3.05 mm to (23.0, 22.4)
- moved C19 0.91 mm to (26.1, 27.5)
Connections:
- new net N$18: J1.P$4, U2.43
- new net N$19: J4.P$4, U2.45
- new net N$20: J1.P$3, U2.47
- new net N$21: J4.P$3, U2.49
- new net N$22: J1.P$2, U2.51
- new net N$23: J4.P$2, U2.53
- new net N$24: J1.P$1, U2.55
- new net N$25: J4.P$1, U2.1
- new net REF_ELEC: J4.P$5, U2.42, U2.44, U2.46, U2.48, U2.50, U2.52, U2.54, U2.56
- net DCDC_SW: now also U$1.33; no longer CC2652R1.33
- net GND: now also J1.P$5, U$1.EGP; no longer CC2652R1.EGP, U2.42, U2.44, U2.46, U2.48, U2.50, U2.52, U2.54, U2.56
- net JTAG_TCK: now also U$1.25; no longer CC2652R1.25
- net JTAG_TDI: now also U$1.27; no longer CC2652R1.27
- net JTAG_TDO: now also U$1.26; no longer CC2652R1.26
- net JTAG_TMS: now also U$1.24; no longer CC2652R1.24
- net N$1: now also U$1.23; no longer CC2652R1.23
- net N$10: now also U$1.4; no longer CC2652R1.4
- net N$13: now also U$1.38; no longer CC2652R1.38
- net N$17: now also U$1.37; no longer CC2652R1.37
- net N$3: now also U$1.47; no longer CC2652R1.47
- net N$4: now also U$1.46; no longer CC2652R1.46
- net N$5: now also U$1.3; no longer CC2652R1.3
- net RF_N: now also U$1.2; no longer CC2652R1.2
- net RF_P: now also U$1.1; no longer CC2652R1.1
- net RXD: now also U$1.7; no longer CC2652R1.7
- net SPI_CLK: now also U$1.16; no longer CC2652R1.16
- net SPI_CS_TP: now also U$1.12; no longer CC2652R1.12
- net SPI_MISO: now also U$1.14; no longer CC2652R1.14
- net SPI_MOSI: now also U$1.15; no longer CC2652R1.15
- net TXD: now also U$1.8; no longer CC2652R1.8
- net VDDR: now also U$1.45, U$1.48; no longer CC2652R1.45, CC2652R1.48
- net VDDS3V3: now also U$1.13, U$1.22, U$1.34, U$1.44; no longer CC2652R1.13, CC2652R1.22, CC2652R1.34, CC2652R1.44
- net WMCU_RESET: now also U$1.35; no longer CC2652R1.35
Routing:
- net REF_ELEC: track 0.00 -> 17.0 mm, vias 0 -> 1
- net VCC: track 45.2 -> 59.9 mm
- net GND: track 138.4 -> 128.7 mm, vias 30 -> 31
- net N$24: track 0.00 -> 7.61 mm
- net N$22: track 0.00 -> 7.22 mm
- net N$20: track 0.00 -> 7.12 mm
- net N$18: track 0.00 -> 7.11 mm
- net N$25: track 0.00 -> 5.04 mm
- net N$23: track 0.00 -> 4.14 mm
- net N$21: track 0.00 -> 3.94 mm
- net SPI_CLK: track 22.5 -> 18.7 mm
- net N$19: track 0.00 -> 3.69 mm
- net SPI_MOSI: track 19.5 -> 17.0 mm
- net SPI_MISO: track 17.2 -> 14.9 mm
- net N$10: track 10.0 -> 10.9 mm
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Other:
- board text added: "10"
- board text added: "11"
- board text added: "4"
- board text added: "5"
- board text added: "6"
- board text added: "7"
- board text added: "8"
- board text added: "9"
